Commit message: Update ur7e_robot.urdf to use local relative mesh paths instead of package:// references

File: assets/ur7e_robot.urdf (robot description, URDF)
Before this commit: robot ur7e_robot, 11 links, 10 joints
Links:
- added link ft_frame
- added link world
- link base_link_inertia: geometry collision mesh filename=meshes/ur5e/collision/base.stl; visual mesh filename=meshes/ur5e/visual/base.dae
- link forearm_link: geometry collision mesh filename=meshes/ur5e/collision/forearm.stl; visual mesh filename=meshes/ur5e/visual/forearm.dae
- link shoulder_link: geometry collision mesh filename=meshes/ur5e/collision/shoulder.stl; visual mesh filename=meshes/ur5e/visual/shoulder.dae
- link upper_arm_link: geometry collision mesh filename=meshes/ur5e/collision/upperarm.stl; visual mesh filename=meshes/ur5e/visual/upperarm.dae
- link wrist_1_link: geometry collision mesh filename=meshes/ur5e/collision/wrist1.stl; visual mesh filename=meshes/ur5e/visual/wrist1.dae
- link wrist_2_link: geometry collision mesh filename=meshes/ur5e/collision/wrist2.stl; visual mesh filename=meshes/ur5e/visual/wrist2.dae
- link wrist_3_link: geometry collision mesh filename=meshes/ur5e/collision/wrist3.stl; visual mesh filename=meshes/ur5e/visual/wrist3.dae
Joints:
- added joint base_joint: type fixed, parent world, child base_link, origin xyz=0 0 0 rpy=0 0 0
- added joint wrist_3_link-ft_frame: type fixed, parent wrist_3_link, child ft_frame, origin xyz=0 0 0 rpy=3.141592653589793 0 0
